File: dsPIC33EV256GM104-PT.kicad_pcb (KiCad board)
At the start: 2 copper layers, 80 x 55 mm, 27 parts, among them P1 POWER, P2 ICSP, P3 CONN_01X09, P4 CONN_01X09, P5 CONN_01X09, P6 CONN_01X09, SW1 RESET, U1 dsPIC33EVxxxGMx04, Y1 Crystal

Commit message: 1.0
Parts:
- D1: value Led_Green -> Green
- L1: value L_Small -> 2,2uH
- P3, P4, P5, P6: value CONN_01X09 -> I/O
Changed lines of the file:
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@@
   )
   (page A4)
+  (title_block
+    (title "dsPIC33EV256GM104 MiniStarter Kit")
+    (date 2015-12-06)
+    (rev 1.0)
+    (company TIETom)
+  )
   (layers
     (0 F.Cu signal hide)
@@
     (visible_elements 7FFFFF7F)
     (pcbplotparams
-      (layerselection 0x00030_80000001)
+      (layerselection 0x00020_00000000)
       (usegerberextensions false)
-      (excludeedgelayer true)
+      (excludeedgelayer false)
       (linewidth 0.100000)
       (plotframeref false)
@@
       (plotvalue true)
       (plotinvisibletext false)
-      (padsonsilk false)
+      (padsonsilk true)
       (subtractmaskfromsilk false)
-      (outputformat 1)
-      (mirror false)
-      (drillshape 1)
+      (outputformat 2)
+      (mirror true)
+      (drillshape 2)
       (scaleselection 1)
       (outputdirectory ""))
@@
       (effects (font (size 1 1) (thickness 0.15)))
     )
-    (fp_text value CONN_01X09 (at 0 -3.1 90) (layer F.Fab) hide
+    (fp_text value I/O (at 0 -3.1 90) (layer F.Fab) hide
       (effects (font (size 1 1) (thickness 0.15)))
     )
@@
     (tags "capacitor 0805")
     (attr smd)
-    (fp_text reference C1 (at 0 2.1) (layer B.SilkS)
-      (effects (font (size 1 1) (thickness 0.15)) (justify mirror))
-    )
-    (fp_text value 100n (at 0 -2.1) (layer B.Fab)
+    (fp_text reference C1 (at 4.175 0) (layer B.SilkS)
+      (effects (font (size 1 1) (thickness 0.15)) (justify mirror))
+    )
+    (fp_text value 100n (at -4.08 0) (layer B.Fab)
       (effects (font (size 1 1) (thickness 0.15)) (justify mirror))
     )
@@
     (tags "capacitor 0603")
     (attr smd)
-    (fp_text reference C2 (at 0 1.9) (layer B.SilkS)
-      (effects (font (size 1 1) (thickness 0.15)) (justify mirror))
-    )
-    (fp_text value 10n (at 0 -1.9) (layer B.Fab)
+    (fp_text reference C2 (at 2.54 0) (layer B.SilkS)
+      (effects (font (size 1 1) (thickness 0.15)) (justify mirror))
+    )
+    (fp_text value 10n (at -3.175 0) (layer B.Fab)
       (effects (font (size 1 1) (thickness 0.15)) (justify mirror))
     )
@@
     (tags "capacitor 0603")
     (attr smd)
-    (fp_text reference C3 (at 0 1.9) (layer B.SilkS)
-      (effects (font (size 1 1) (thickness 0.15)) (justify mirror))
-    )
-    (fp_text value 1n (at 0 -1.9) (layer B.Fab)
+    (fp_text reference C3 (at 2.54 0) (layer B.SilkS)
+      (effects (font (size 1 1) (thickness 0.15)) (justify mirror))
+    )
+    (fp_text value 1n (at -2.54 0) (layer B.Fab)
       (effects (font (size 1 1) (thickness 0.15)) (justify mirror))
     )
@@
     (tags "Tantal Capacitor Size-C EIA-6032 Reflow")
     (attr smd)
-    (fp_text reference C5 (at -0.1 2.7) (layer B.SilkS)
+    (fp_text reference C5 (at 0 -4.445) (layer B.SilkS)
       (effects (font (size 1 1) (thickness 0.15)) (justify mirror))
     )
@@
     (tags "capacitor 0805")
     (attr smd)
-    (fp_text reference C6 (at 0 2.1) (layer B.SilkS)
-      (effects (font (size 1 1) (thickness 0.15)) (justify mirror))
-    )
-    (fp_text value 100n (at 0 -2.1) (layer B.Fab)
+    (fp_text reference C6 (at 3.445 0) (layer B.SilkS)
+      (effects (font (size 1 1) (thickness 0.15)) (justify mirror))
+    )
+    (fp_text value 100n (at -4.175 0) (layer B.Fab)
       (effects (font (size 1 1) (thickness 0.15)) (justify mirror))
     )
@@
     (tags "capacitor 0805")
     (attr smd)
-    (fp_text reference C7 (at 0 2.1 180) (layer B.SilkS)
-      (effects (font (size 1 1) (thickness 0.15)) (justify mirror))
-    )
-    (fp_text value 100n (at 0 -2.1 180) (layer B.Fab)
+    (fp_text reference C7 (at -3.81 0 180) (layer B.SilkS)
+      (effects (font (size 1 1) (thickness 0.15)) (justify mirror))
+    )
+    (fp_text value 100n (at -3.81 -1.27 180) (layer B.Fab)
       (effects (font (size 1 1) (thickness 0.15)) (justify mirror))
     )
@@
     (tags "capacitor 0603")
     (attr smd)
-    (fp_text reference C8 (at 0 1.9) (layer B.SilkS)
-      (effects (font (size 1 1) (thickness 0.15)) (justify mirror))
-    )
-    (fp_text value 10n (at 0 -1.9) (layer B.Fab)
+    (fp_text reference C8 (at 3.06 0) (layer B.SilkS)
+      (effects (font (size 1 1) (thickness 0.15)) (justify mirror))
+    )
+    (fp_text value 10n (at -3.29 0) (layer B.Fab)
       (effects (font (size 1 1) (thickness 0.15)) (justify mirror))
     )
@@
     (tags "capacitor 0603")
     (attr smd)
-    (fp_text reference C9 (at 0 1.9 180) (layer B.SilkS)
-      (effects (font (size 1 1) (thickness 0.15)) (justify mirror))
-    )
-    (fp_text value 10n (at 0 -1.9 180) (layer B.Fab)
+    (fp_text reference C9 (at -3.81 0 180) (layer B.SilkS)
+      (effects (font (size 1 1) (thickness 0.15)) (justify mirror))
+    )
+    (fp_text value 10n (at -3.81 -1.27 180) (layer B.Fab)
       (effects (font (size 1 1) (thickness 0.15)) (justify mirror))
     )
@@
     (tags "capacitor 0603")
     (attr smd)
-    (fp_text reference C10 (at 0 1.9) (layer B.SilkS)
-      (effects (font (size 1 1) (thickness 0.15)) (justify mirror))
-    )
-    (fp_text value 1n (at 0 -1.9) (layer B.Fab)
+    (fp_text reference C10 (at 3.175 0) (layer B.SilkS)
+      (effects (font (size 1 1) (thickness 0.15)) (justify mirror))
+    )
+    (fp_text value 1n (at -2.54 0) (layer B.Fab)
       (effects (font (size 1 1) (thickness 0.15)) (justify mirror))
     )
@@
     (tags "capacitor 0603")
     (attr smd)
-    (fp_text reference C11 (at 0 1.9 180) (layer B.SilkS)
-      (effects (font (size 1 1) (thickness 0.15)) (justify mirror))
-    )
-    (fp_text value 1n (at 0 -1.9 180) (layer B.Fab)
+    (fp_text reference C11 (at -3.06 1.27 180) (layer B.SilkS)
+      (effects (font (size 1 1) (thickness 0.15)) (justify mirror))
+    )
+    (fp_text value 1n (at -3.06 0 180) (layer B.Fab)
       (effects (font (size 1 1) (thickness 0.15)) (justify mirror))
     )
@@
       (effects (font (size 1 1) (thickness 0.15)))
     )
-    (fp_text value C_Crystal (at 1.25 2.5 225) (layer F.Fab)
+    (fp_text value C_Crystal (at 1.152962 -4.041115 225) (layer F.Fab)
       (effects (font (size 1 1) (thickness 0.15)))
     )
@@
       (effects (font (size 1 1) (thickness 0.15)))
     )
-    (fp_text value C_Crystal (at 1.25 2.5 45) (layer F.Fab)
+    (fp_text value C_Crystal (at 8.082231 0 45) (layer F.Fab)
       (effects (font (size 1 1) (thickness 0.15)))
     )
@@
       (effects (font (size 1 1) (thickness 0.15)))
     )
-    (fp_text value Led_Green (at 1.524 -3.937 90) (layer F.Fab)
+    (fp_text value Green (at -2.54 0 180) (layer F.Fab)
       (effects (font (size 1 1) (thickness 0.15)))
     )
@@
     (descr "Resistor, SMD and THT, universal, 0805 to 1206,RM10,  Hand soldering,")
     (tags "Resistor, SMD and THT, universal, 0805 to 1206, RM10, Hand soldering,")
-    (fp_text reference L1 (at 0.09906 3.0988 180) (layer B.SilkS) hide
-      (effects (font (size 1 1) (thickness 0.15)) (justify mirror))
-    )
-    (fp_text value L_Small (at -0.39878 -4.20116 180) (layer B.Fab) hide
-      (effects (font (size 1 1) (thickness 0.15)) (justify mirror))
+    (fp_text reference L1 (at 0 -3.175 180) (layer F.SilkS)
+      (effects (font (size 1 1) (thickness 0.15)))
+    )
+    (fp_text value 2,2uH (at 0 -5.08 180) (layer F.Fab)
+      (effects (font (size 1 1) (thickness 0.15)))
     )
     (fp_line (start 0 -0.8001) (end 0.20066 -0.8001) (layer B.SilkS) (width 0.15))
@@
       (effects (font (size 1 1) (thickness 0.15)))
     )
-    (fp_text value CONN_01X09 (at 0 -3.1 90) (layer F.Fab) hide
+    (fp_text value I/O (at 0 -3.1 90) (layer F.Fab) hide
       (effects (font (size 1 1) (thickness 0.15)))
     )
@@
       (effects (font (size 1 1) (thickness 0.15)))
     )
-    (fp_text value CONN_01X09 (at 0 -3.1 270) (layer F.Fab) hide
+    (fp_text value I/O (at 0 -3.1 270) (layer F.Fab) hide
       (effects (font (size 1 1) (thickness 0.15)))
     )
@@
       (effects (font (size 1 1) (thickness 0.15)))
     )
-    (fp_text value CONN_01X09 (at 0 -3.1 270) (layer F.Fab) hide
+    (fp_text value I/O (at 0 -3.1 270) (layer F.Fab) hide
       (effects (font (size 1 1) (thickness 0.15)))
     )
@@
       (effects (font (size 1 1) (thickness 0.15)) (justify mirror))
     )
-    (fp_text value 1k (at 0 -2.1) (layer B.Fab)
+    (fp_text value 1k (at 0 3.81) (layer B.Fab)
       (effects (font (size 1 1) (thickness 0.15)) (justify mirror))
     )
@@
     (tags "resistor 0805")
     (attr smd)
-    (fp_text reference R2 (at 0 2.1 180) (layer B.SilkS)
-      (effects (font (size 1 1) (thickness 0.15)) (justify mirror))
-    )
-    (fp_text value 10k (at 0 -2.1 180) (layer B.Fab)
-      (effects (font (size 1 1) (thickness 0.15)) (justify mirror))
-    )
+    (fp_text reference R2 (at 0 3.175 180) (layer B.SilkS)
+      (effects (font (size 1 1) (thickness 0.15)) (justify mirror))
+    )
+    (fp_text value 10k (at 0 1.905 180) (layer B.Fab)
+      (effects (font (size 1 1) (thickness 0.15)) (justify mirror))
+    )
