File: dsPIC33EV256GM104-PT.sch (KiCad schematic (older format))
At the start: 26 parts, among them P1 POWER, P2 ICSP, P3 CONN_01X09, P4 CONN_01X09, P5 CONN_01X09, P6 CONN_01X09, SW1 RESET, U1 dsPIC33EVxxxGMx04, Y1 Crystal

Commit message: 1.0
Parts:
- D1: value Led_Green -> Green
- L1: value L_Small -> 2,2uH
- P3, P4, P5, P6: value CONN_01X09 -> I/O
Other:
- note added: "I/O"
- note added: "ICSP"
- note added: "MICROCONTROLER"
- note added: "POWER"
- note added: "RESET\n"
- moved on the sheet: C1, C10, C11, C12, C13, C2, C3, C4, C5, C6, C7, C8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
